File: stlink-swd.sch (KiCad schematic (older format))
At the start: 7 parts, among them J1 Conn_02x03_Odd_Even, J2 Ribbon IDC DIP, J3 SWD-RA, J4 Conn_01x02, SW1 KS-00Q-02

Commit message: Added part numbers and rounded PCB edges
Also deleted some temporary BOM files that got checked in.
Parts:
- D1: Part No. (none) -> 732-4980-1-ND
- J1: Part No. (none) -> S2012EC-03-ND
- J4: Part No. (none) -> S1012EC-02-ND
Other:
- note added: "Jumper: S9337-ND"
Changed lines of the file:
@@
 F 2 "Pin_Headers:Pin_Header_Straight_2x03_Pitch2.54mm" H 5450 3300 50  0001 C CNN
 F 3 "~" H 5450 3300 50  0001 C CNN
+F 4 "S2012EC-03-ND" H 5450 3300 50  0001 C CNN "Part No."
 	1    5450 3300
 	-1   0    0    -1
@@
 F 2 "Pin_Headers:Pin_Header_Straight_1x02_Pitch2.54mm" H 5500 3900 50  0001 C CNN
 F 3 "~" H 5500 3900 50  0001 C CNN
+F 4 "S1012EC-02-ND" H 5500 3900 50  0001 C CNN "Part No."
 	1    5500 3900
 	-1   0    0    -1
@@
 F 2 "LEDs:LED_0603" H 6200 4350 50  0001 C CNN
 F 3 "~" H 6200 4350 50  0001 C CNN
+F 4 "732-4980-1-ND" H 6200 4350 50  0001 C CNN "Part No."
 	1    6200 4350
 	0    -1   -1   0
@@
 	5000 3300 5150 3300
 Connection ~ 4550 3400
+Text Notes 5050 2850 0    50   ~ 0
+Jumper: S9337-ND
 $EndSCHEMATC
